File: microcontroller.kicad_sch (KiCad schematic)
At the start: 15 parts, among them J11 ESP32 [R], J16 ESP32 [L], U12 DHT20, U2 M24C02-FMN, U5 DIO5661ST6

Commit message: Maintenance update - Adding the EC isolation board schematic - Added a harness page for wireing module together
Parts:
- C1, C26: MPN (none) -> CC0805KRX7R7BB104; Manufacturer (none) -> YAGEO; Package (none) -> 0805
- C18: MPN (none) -> CL21B105KOFNNNG; Manufacturer (none) -> Samsung; Package (none) -> 0805
- C29: MPN (none) -> CL21B106KPQNNNE; Manufacturer (none) -> Samsung; Package (none) -> 0805
- C37: MPN (none) -> CL21B474KOFNNNE; Manufacturer (none) -> Samsung; Package (none) -> 0805
- D5: MPN (none) -> B230-13-F; Manufacturer (none) -> Diodes Inc.; Package (none) -> SMB
- J11, J16, U12: now not fitted
- L2: MPN (none) -> CBC3225T220KR; Manufacturer (none) -> Tayo Yuden; Package (none) -> 1210
- R27: MPN (none) -> AC0805FR-7W10RL; Manufacturer (none) -> YAGEO; Package (none) -> 0805
- R33, R34: MPN (none) -> AC0805FR-7W4K7L; Manufacturer (none) -> YAGEO; Package (none) -> 0805
- U2: MPN (none) -> M24C02-FMN; Manufacturer (none) -> ST; Package (none) -> SOIC-8
- U5: MPN (none) -> DIO5661ST6; Manufacturer (none) -> DIOO; Package (none) -> SOT-23-6
Other:
- note added: "BUG: Audit the strapping pins. When attached to the board, the ESP32 module boots in a protected mode. This may be due to the strapping pins being held low. Possibly GPIO_0 is the culprit. Add a pullup or pulldown where appropriate on these pins for proper booting."
