File: power.kicad_sch (KiCad schematic)
At the start: 48 parts, among them U11 OPA197xDGK, U13 TLV4387, U14 MCP1727-5002xSN, U16 AP63200WU, U6 TPS22929D, U7 REF3040, U8 REF3025

Commit message: BUG FIX -------- There were some issues with the board WRT manufacturing. I changed the VSSOP 8 packages to SOT versions and re-routed
Parts:
- removed U11: OPA197xDGK, Package_SO:VSSOP-8_3x3mm_P0.65mm, symbol Amplifier_Operational:OPA197xDGK
- added U3: OPA197xD, Package_SO:SOIC-8_3.9x4.9mm_P1.27mm, symbol Amplifier_Operational:OPA197xD
Connections:
- net INPUT_COMMON: now also U3.4 (V-)
- net INPUT_VBATT_+: now also U3.7 (V+)
- net at R30.2, R32.1: now also U3.2 (-)
- net at R32.2, R38.1: now also U3.6
- net at R29.2, R31.1: now also U3.3 (+)
Changed lines of the file:
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@@
 	)
 	(junction
-		(at 238.76 81.28)
-		(diameter 0)
-		(color 0 0 0 0)
-	)
-	(junction
 		(at 120.65 36.83)
 		(diameter 0)
@@
 	)
 	(junction
+		(at 238.76 81.28)
+		(diameter 0)
+		(color 0 0 0 0)
+	)
+	(junction
 		(at 72.39 26.67)
 		(diameter 0)
@@
 	(wire
 		(pts
-			(xy 240.03 140.97) (xy 240.03 146.05)
-		)
-		(stroke
-			(width 0)
-			(type default)
-		)
-	)
-	(wire
-		(pts
 			(xy 100.33 36.83) (xy 100.33 31.75)
 		)
@@
 		)
 	)
-	(hierarchical_label "+4.096_REF_BUF_A"
-		(shape output)
-		(at 240.03 146.05 270)
-		(effects
-			(font
-				(size 1.27 1.27)
-			)
-			(justify right)
-		)
-	)
 	(hierarchical_label "DIGITAL_GND"
 		(shape output)
@@
 	)
 	(symbol
-		(lib_id "Amplifier_Operational:OPA197xDGK")
-		(at 231.14 81.28 0)
-		(unit 1)
-		(exclude_from_sim no)
-		(in_bom yes)
-		(on_board yes)
-		(dnp no)
-		(property "Reference" "U11"
-			(at 232.156 71.628 0)
-			(effects
-				(font
-					(size 1.27 1.27)
-				)
-			)
-		)
-		(property "Value" "OPA197xDGK"
-			(at 236.22 73.914 0)
-			(effects
-				(font
-					(size 1.27 1.27)
-				)
-			)
-		)
-		(property "Footprint" "Package_SO:VSSOP-8_3x3mm_P0.65mm"
-			(at 231.14 81.28 0)
-			(effects
-				(font
-					(size 1.27 1.27)
-				)
-				(hide yes)
-			)
-		)
-		(property "Datasheet" "http://www.ti.com/lit/ds/symlink/opa197.pdf"
-			(at 231.14 76.2 0)
-			(effects
-				(font
-					(size 1.27 1.27)
-				)
-				(hide yes)
-			)
-		)
-		(property "Description" "Single 36V, Precision, Rail-to-Rail Input/Output, Low Offset Voltage, Operational Amplifier, VSSOP-8"
-			(at 231.14 81.28 0)
-			(effects
-				(font
-					(size 1.27 1.27)
-				)
-				(hide yes)
-			)
-		)
-		(pin "7"
-		)
-		(pin "2"
-		)
-		(pin "3"
-		)
-		(pin "5"
-		)
-		(pin "8"
-		)
-		(pin "1"
-		)
-		(pin "6"
-		)
-		(pin "4"
-		)
-		(instances
-			(project ""
-				(path "/37fdfe07-1a70-41c8-8af2-e03e19737580/1fb5cba5-fe5a-4aba-b82b-13cd9370505b"
-					(reference "U11")
-					(unit 1)
-				)
-			)
-		)
-	)
-	(symbol
 		(lib_id "Device:R")
 		(at 129.54 125.73 0)
@@
 	)
 	(symbol
-		(lib_id "power:PWR_FLAG")
-		(at 240.03 140.97 0)
-		(unit 1)
-		(exclude_from_sim no)
-		(in_bom yes)
-		(on_board yes)
-		(dnp no)
-		(fields_autoplaced yes)
-		(property "Reference" "#FLG8"
-			(at 240.03 139.065 0)
-			(effects
-				(font
-					(size 1.27 1.27)
-				)
-				(hide yes)
-			)
-		)
-		(property "Value" "PWR_FLAG"
-			(at 240.03 135.89 0)
-			(effects
-				(font
-					(size 1.27 1.27)
-				)
-			)
-		)
-		(property "Footprint" ""
-			(at 240.03 140.97 0)
-			(effects
-				(font
-					(size 1.27 1.27)
-				)
-				(hide yes)
-			)
-		)
-		(property "Datasheet" "~"
-			(at 240.03 140.97 0)
-			(effects
-				(font
-					(size 1.27 1.27)
-				)
-				(hide yes)
-			)
-		)
-		(property "Description" "Special symbol for telling ERC where power comes from"
-			(at 240.03 140.97 0)
-			(effects
-				(font
-					(size 1.27 1.27)
-				)
-				(hide yes)
-			)
-		)
-		(pin "1"
-		)
-		(instances
-			(project "digital_waters"
-				(path "/37fdfe07-1a70-41c8-8af2-e03e19737580/1fb5cba5-fe5a-4aba-b82b-13cd9370505b"
-					(reference "#FLG8")
-					(unit 1)
-				)
-			)
-		)
-	)
-	(symbol
 		(lib_id "Device:C")
 		(at 66.04 181.61 0)
@@
 					(unit 1)
 				)
+			)
+		)
+	)
+	(symbol
+		(lib_id "Amplifier_Operational:OPA197xD")
+		(at 231.14 81.28 0)
+		(unit 1)
+		(exclude_from_sim no)
+		(in_bom yes)
+		(on_board yes)
+		(dnp no)
+		(property "Reference" "U3"
+			(at 232.918 74.676 0)
+			(effects
+				(font
+					(size 1.27 1.27)
+				)
+			)
+		)
+		(property "Value" "OPA197xD"
+			(at 236.22 77.216 0)
+			(effects
+				(font
+					(size 1.27 1.27)
+				)
+			)
+		)
+		(property "Footprint" "Package_SO:SOIC-8_3.9x4.9mm_P1.27mm"
+			(at 228.6 86.36 0)
+			(effects
+				(font
+					(size 1.27 1.27)
+				)
+				(justify left)
+				(hide yes)
+			)
+		)
+		(property "Datasheet" "http://www.ti.com/lit/ds/symlink/opa197.pdf"
+			(at 234.95 77.47 0)
+			(effects
+				(font
+					(size 1.27 1.27)
+				)
+				(hide yes)
+			)
+		)
+		(property "Description" "Single 36V, Precision, Rail-to-Rail Input/Output, Low Offset Voltage, Operational Amplifier, SOIC-8"
+			(at 231.14 81.28 0)
+			(effects
+				(font
+					(size 1.27 1.27)
+				)
+				(hide yes)
+			)
+		)
+		(pin "5"
+		)
+		(pin "4"
+		)
+		(pin "1"
+		)
+		(pin "2"
+		)
+		(pin "7"
+		)
+		(pin "6"
+		)
+		(pin "8"
+		)
+		(pin "3"
+		)
+		(instances
+			(project ""
+				(path "/37fdfe07-1a70-41c8-8af2-e03e19737580/1fb5cba5-fe5a-4aba-b82b-13cd9370505b"
+					(reference "U3")
+					(unit 1)
+				)

Commit message: Maintenance update - Adding the EC isolation board schematic - Added a harness page for wireing module together
Parts:
- removed R4: 0 Ohm, Resistor_SMD:R_1206_3216Metric_Pad1.30x1.75mm_HandSolder, symbol Device:R
- C10: value 100nF -> 0.1u; MPN (none) -> CC0805KRX7R7BB104; Manufacturer (none) -> YAGEO; Package (none) -> 0805
- C11, C14: MPN (none) -> GRM21BZ71A226ME15L; Manufacturer (none) -> Murata; Package (none) -> 0805
- C12, C20, C27, C28, C39, C40, C8: MPN (none) -> CL21B105KOFNNNG; Manufacturer (none) -> Samsung; Package (none) -> 0805
- C13, C16, C19, C21, C22: MPN (none) -> CC0805KRX7R7BB104; Manufacturer (none) -> YAGEO; Package (none) -> 0805
- C15, C7: MPN (none) -> CL21B106KPQNNNE; Manufacturer (none) -> Samsung; Package (none) -> 0805
- C30, C36: MPN (none) -> CL21B474KOFNNNE; Manufacturer (none) -> Samsung; Package (none) -> 0805
- C38: MPN (none) -> C0805C101M4RACTU; Manufacturer (none) -> KEMET; Package (none) -> 0805
- C6: MPN (none) -> CC0805KKX7R7BB824; Manufacturer (none) -> YAGEO; Package (none) -> 0805
- C9: value 10uF -> 10u; MPN (none) -> CL21B106KPQNNNE; Manufacturer (none) -> Samsung; Package (none) -> 0805
- D1, D2, D3: MPN (none) -> LTST-C170GKT; Manufacturer (none) -> Lite-On; Package (none) -> 0805
- D4, D6: MPN (none) -> B230-13-F; Manufacturer (none) -> Diodes Inc.; Package (none) -> SMB
- D8: MPN (none) -> PTVS22VZ1USK; Manufacturer (none) -> Nexperia; Package (none) -> DSN1608-2
- L1: MPN (none) -> DFE322512F-3R3M=P2; Manufacturer (none) -> Murata; Package (none) -> 1210
- R13, R9: MPN (none) -> RCC0805470RFKEA; Manufacturer (none) -> Vishay-Dale; Package (none) -> 0805
- R15: MPN (none) -> RK73H2ATTD6202F; Manufacturer (none) -> KOA Speer Electronics, Inc.; Package (none) -> 0805
- R16, R29, R30: MPN (none) -> AC0805FR-7W10KL; Manufacturer (none) -> YAGEO; Package (none) -> 0805
- R28: MPN (none) -> PE1206FRF7W0R1L; Manufacturer (none) -> YAGEO; Package (none) -> 1206
- R31, R32: MPN (none) -> AC0805FR-7W100KL; Manufacturer (none) -> YAGEO; Package (none) -> 0805
- R38: MPN (none) -> AC0805FR-7W1KL; Manufacturer (none) -> YAGEO; Package (none) -> 0805
- R5: value 2k -> 2.2k; MPN (none) -> AC0805FR-7W2K2L; Manufacturer (none) -> YAGEO; Package (none) -> 0805
- U13: MPN (none) -> TLV4387PWR; Manufacturer (none) -> TI; Package (none) -> TSSOP-14
- U14: MPN (none) -> MCP1727-5002E/SN; Manufacturer (none) -> Microchip; Package (none) -> SOIC-8
- U16: MPN (none) -> AP63200WU-7; Package (none) -> TSOT-26
- U3: MPN (none) -> OPA197ID; Manufacturer (none) -> TI; Package (none) -> SOIC-8
- U6: MPN (none) -> TPS22929DDBVR; Manufacturer (none) -> TI; Package (none) -> SOT-23-6
- U7: MPN (none) -> REF3040AIDBZR; Manufacturer (none) -> TI; Package (none) -> SOT-23
- U8: MPN (none) -> REF3025AIDBZR; Manufacturer (none) -> TI; Package (none) -> SOT-23
Other:
- note added: "BUG: ABS max Vin for the MCP1727 is 6.5 V. I want to use a 7.4V battery. Need a better solution here."
- note added: "BUG: Add overvoltge (6V) protection Zener here"
- note added: "BUG: Remove current shunt. Move this to the battery module."
- note added: "BUG: Spec actual voltage limits here (The AP63200 can go as high as 32V)"
- note added: "BUG: These are wrong"
- note added: "ERC overrides"
- note added: "TODO: - Add a MOV - Add reverse voltage protection"
- note removed: "AGND and DGND are tied together internally to the MCP320X. This connection should be as close to thay chip as possible."
- note removed: "TODO: Add a MOV"
