File: power.kicad_sch (KiCad schematic)
At the start: 48 parts, among them U13 TLV4387, U14 MCP1727-5002xSN, U16 AP63200WU, U3 OPA197xD, U6 TPS22929D, U7 REF3040, U8 REF3025

Commit message: feature/v3.1/setup - Inception - some general changes in support of v3.1 before I thought to branch.
Parts:
- removed C16, C19, C21, C22: 0.1u, Capacitor_SMD:C_0805_2012Metric_Pad1.18x1.45mm_HandSolder, symbol Device:C
- removed C20, C27, C28, C8: 1u, Capacitor_SMD:C_0805_2012Metric_Pad1.18x1.45mm_HandSolder, symbol Device:C
- removed R28: 0.1 / 1% / 0.5W / Metal Film, Resistor_SMD:R_1206_3216Metric_Pad1.30x1.75mm_HandSolder, symbol Device:R
- removed R4: 0 Ohm, Resistor_SMD:R_1206_3216Metric_Pad1.30x1.75mm_HandSolder, symbol Device:R
- C10: value 100nF -> 0.1u; MPN (none) -> CC0805KRX7R7BB104; Manufacturer (none) -> YAGEO; Package (none) -> 0805
- C11, C14: MPN (none) -> GRM21BZ71A226ME15L; Manufacturer (none) -> Murata; Package (none) -> 0805
- C12, C39, C40: MPN (none) -> CL21B105KOFNNNG; Manufacturer (none) -> Samsung; Package (none) -> 0805
- C13: MPN (none) -> CC0805KRX7R7BB104; Manufacturer (none) -> YAGEO; Package (none) -> 0805
- C15, C7: MPN (none) -> CL21B106KPQNNNE; Manufacturer (none) -> Samsung; Package (none) -> 0805
- C30, C36: MPN (none) -> CL21B474KOFNNNE; Manufacturer (none) -> Samsung; Package (none) -> 0805
- C38: MPN (none) -> C0805C101M4RACTU; Manufacturer (none) -> KEMET; Package (none) -> 0805
- C6: MPN (none) -> CC0805KKX7R7BB824; Manufacturer (none) -> YAGEO; Package (none) -> 0805; now not fitted; now left out of the parts list
- C9: value 10uF -> 10u; MPN (none) -> CL21B106KPQNNNE; Manufacturer (none) -> Samsung; Package (none) -> 0805
- D1, D2, D3: MPN (none) -> LTST-C170GKT; Manufacturer (none) -> Lite-On; Package (none) -> 0805
- D4, D6: MPN (none) -> B230-13-F; Manufacturer (none) -> Diodes Inc.; Package (none) -> SMB
- D8: MPN (none) -> PTVS22VZ1USK; Manufacturer (none) -> Nexperia; Package (none) -> DSN1608-2
- L1: MPN (none) -> DFE322512F-3R3M=P2; Manufacturer (none) -> Murata; Package (none) -> 1210
- R13, R9: MPN (none) -> RCC0805470RFKEA; Manufacturer (none) -> Vishay-Dale; Package (none) -> 0805
- R15: MPN (none) -> RK73H2ATTD6202F; Manufacturer (none) -> KOA Speer Electronics, Inc.; Package (none) -> 0805
- R16: MPN (none) -> AC0805FR-7W10KL; Manufacturer (none) -> YAGEO; Package (none) -> 0805
- R29, R30: MPN (none) -> AC0805FR-7W10KL; Manufacturer (none) -> YAGEO; Package (none) -> 0805; now not fitted; now left out of the parts list
- R31, R32: MPN (none) -> AC0805FR-7W100KL; Manufacturer (none) -> YAGEO; Package (none) -> 0805; now not fitted; now left out of the parts list
- R38: MPN (none) -> AC0805FR-7W1KL; Manufacturer (none) -> YAGEO; Package (none) -> 0805; now not fitted; now left out of the parts list
- R5: value 2k -> 2.2k; MPN (none) -> AC0805FR-7W2K2L; Manufacturer (none) -> YAGEO; Package (none) -> 0805
- U13: MPN (none) -> TLV4387PWR; Manufacturer (none) -> TI; Package (none) -> TSSOP-14
- U14: MPN (none) -> MCP1727-5002E/SN; Manufacturer (none) -> Microchip; Package (none) -> SOIC-8
- U16: MPN (none) -> AP63200WU-7; Package (none) -> TSOT-26
- U3: MPN (none) -> OPA197ID; Manufacturer (none) -> TI; Package (none) -> SOIC-8; now not fitted; now left out of the parts list
- U6: MPN (none) -> TPS22929DDBVR; Manufacturer (none) -> TI; Package (none) -> SOT-23-6
- U7: MPN (none) -> REF3040AIDBZR; Manufacturer (none) -> TI; Package (none) -> SOT-23
- U8: MPN (none) -> REF3025AIDBZR; Manufacturer (none) -> TI; Package (none) -> SOT-23
Connections:
- net +2.5V_REF_BUF_A: now also U13.9 (-); no longer U13.10 (+)
- net +2.5V_REF_BUF_B: now also U13.13 (-); no longer U13.12 (+)
- net DIGITAL_GND: now also C11.2, C14.2, C39.2, C7.1, C9.2, D1.1 (K), D8.2 (A), R16.2, R31.2, U16.4 (GND), U3.4 (V-); no longer R29.1
- removed net INPUT_COMMON: C11.2, C14.2, C39.2, C7.1, C9.2, D1.1 (K), D8.2 (A), R16.2, R30.1, R31.2, U16.4 (GND), U3.4 (V-)
- new net: U13.10 (+), U13.12 (+), U8.2 (OUT)
Other:
- added sheet RTC (rtc.kicad_sch)
- note added: "BUG: ABS max Vin for the MCP1727 is 6.5 V. I want to use a 7.4V battery. Need a better solution here."
- note added: "BUG: Add overvoltge (6V) protection Zener here"
- note added: "BUG: Remove current shunt. Move this to the battery module."
- note added: "BUG: Spec actual voltage limits here (The AP63200 can go as high as 32V)"
- note added: "ERC overrides"
- note added: "TODO: - Add a MOV - Add reverse voltage protection"
- note added: "change to 512mV"
- note removed: "AGND and DGND are tied together internally to the MCP320X. This connection should be as close to thay chip as possible."
- note removed: "Reference Decoupling"
- note removed: "TODO: Add a MOV"
- moved on the sheet: C12, C13, C15, C30, C36, C39, C40, C7, D2, D3, R13, R9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
