File: digital_waters.kicad_pcb (KiCad board)
At the start: 4 copper layers, 100 x 45 mm, 118 parts, among them J1 Conn_Batt, J11 ESP32 [R], J16 ESP32 [L], J18 EZO Carrier Board, J2 Conn_Remote, J3 Conn_Sense_A, J4 Conn_Sense_B, J5 Conn_Illum, J6 Cal_in, U1 MCP3208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

Commit message: feature/v3.1/setup - Inception - some general changes in support of v3.1 before I thought to branch.
Parts:
- removed C16, C19, C21, C22: 0.1u, Capacitor_SMD:C_0805_2012Metric_Pad1.18x1.45mm_HandSolder
- removed C20, C27, C28, C8: 1u, Capacitor_SMD:C_0805_2012Metric_Pad1.18x1.45mm_HandSolder
- removed C3, C6: 800n, Capacitor_SMD:C_0805_2012Metric_Pad1.18x1.45mm_HandSolder
- removed R10, R7: 1k / 1%, Resistor_SMD:R_0805_2012Metric_Pad1.20x1.40mm_HandSolder
- removed R17, R21: 10k/1%, Resistor_SMD:R_0805_2012Metric_Pad1.20x1.40mm_HandSolder
- removed R23, R35: 27k/1%, Resistor_SMD:R_0805_2012Metric_Pad1.20x1.40mm_HandSolder
- removed R28: 0.1 / 1% / 0.5W / Metal Film, Resistor_SMD:R_1206_3216Metric_Pad1.30x1.75mm_HandSolder
- removed R29, R30: 10k / 1%, Resistor_SMD:R_0805_2012Metric_Pad1.20x1.40mm_HandSolder
- removed R31, R32: 100k / 1%, Resistor_SMD:R_0805_2012Metric_Pad1.20x1.40mm_HandSolder
- removed R37, R38: 1k, Resistor_SMD:R_0805_2012Metric_Pad1.20x1.40mm_HandSolder
- removed U3: OPA197xD, Package_SO:SOIC-8_3.9x4.9mm_P1.27mm
- C10: value 100nF -> 0.1u
- C9: value 10uF -> 10u
- R25: value 96k / 1% -> 91k / 1%
- R5: value 2k -> 2.2k
- moved R13 31.2 mm to (197.5, 140.0)
- moved U7 31.2 mm to (186.9, 145.9)
- moved C12 31.2 mm to (195.1, 141.2)
- moved C13 31.2 mm to (192.8, 141.2)
- moved C36 31.2 mm to (202.1, 144.0)
- moved C40 31.2 mm to (209.9, 134.2)
- moved D3 31.2 mm to (194.9, 136.2)
- moved U13 31.2 mm to (193.9, 147.0)
- moved U6 31.2 mm to (206.4, 134.3)
- moved U8 31.2 mm to (202.0, 147.0)
- moved C30 31.2 mm to (186.9, 148.8)
Connections:
- C11 pad 2: /Power/INPUT_COMMON -> GNDD
- C14 pad 2: /Power/INPUT_COMMON -> GNDD
- C39 pad 2: /Power/INPUT_COMMON -> GNDD
- C7 pad 1: /Power/INPUT_COMMON -> GNDD
- C9 pad 2: /Power/INPUT_COMMON -> GNDD
- D1 pad 1: /Power/INPUT_COMMON -> GNDD
- D8 pad 2: /Power/INPUT_COMMON -> GNDD
- J1 pad 2: /Power/INPUT_COMMON -> GNDD
- J2 pad 3: /Power/INPUT_COMMON -> GNDD
- R16 pad 2: /Power/INPUT_COMMON -> GNDD
- R4 pad 1: GNDD -> /DIGITAL_GND
- R4 pad 2: GNDA -> /ANALOG_GND
- U13 pad 10: /Power/+2.5V_REF_BUF_A -> Net-(U13C-+)
- U13 pad 12: /Power/+2.5V_REF_BUF_B -> Net-(U13C-+)
- U13 pad 13: Net-(U13C--) -> /Power/+2.5V_REF_BUF_B
- U13 pad 9: Net-(U13C--) -> /Power/+2.5V_REF_BUF_A
- U16 pad 4: /Power/INPUT_COMMON -> GNDD
- U8 pad 2: Net-(U13C--) -> Net-(U13C-+)
Routing:
- net /Power/+2.5V_REF_BUF_B: track 78.3 -> 13.9 mm
- net /Power/+2.5V_REF_BUF_A: track 65.5 -> 4.86 mm
- net /Power/+4.096_REF_BUF_B: track 58.0 -> 14.5 mm
- net Net-(R32-Pad2): track 28.0 -> 0.00 mm
- net /Micocontroller/ADC_ISENSE: track 18.8 -> 0.00 mm, vias 1 -> 0
- net +VSW: track 50.6 -> 32.0 mm, vias 10 -> 7
- net /Sensor Module Prototype/INPUT_PT1000+: track 18.3 -> 0.00 mm
- net /ADC_VREF: track 17.7 -> 0.00 mm, vias 4 -> 0
- net GNDA: track 65.6 -> 52.1 mm, vias 29 -> 20
- net Net-(U3-+): track 12.7 -> 0.00 mm
- net /Sensor Module Prototype/INPUT_PT1000-: track 10.9 -> 0.00 mm
- net Net-(U13C--): track 8.80 -> 0.00 mm
- net /Power/INPUT_COMMON: track 8.75 -> 0.00 mm, vias 14 -> 0
- net Net-(U13A-+): track 7.04 -> 0.00 mm
- net Net-(U9B--): track 6.64 -> 0.00 mm
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- added copper zone on In1.Cu, net GNDD
- removed copper zone on F.Cu, net /Power/INPUT_COMMON
- removed copper zone on In1.Cu, net /Power/INPUT_COMMON
