File: digital_waters.kicad_sch (KiCad schematic)
At the start: 13 parts, among them J1 Conn_Batt, J2 Conn_Remote, J3 Conn_Sense_A, J4 Conn_Sense_B, J5 Conn_Illum, U1 MCP3208, U10 ST485E

Commit message: feature/v3.1/setup - Inception - some general changes in support of v3.1 before I thought to branch.
Parts:
- added R4: 0 Ohm, Resistor_SMD:R_1206_3216Metric_Pad1.30x1.75mm_HandSolder, symbol Device:R
- C33, C35: MPN (none) -> CL21B105KOFNNNG; Manufacturer (none) -> Samsung; Package (none) -> 0805
- C34: MPN (none) -> CL21B106KPQNNNE; Manufacturer (none) -> Samsung; Package (none) -> 0805
- D7, D9: MPN (none) -> PTVS10VZ1USK; Manufacturer (none) -> Nexperia; Package (none) -> DSN1608-2
- J1, J2, J3, J4, J5: now not fitted
- R14: MPN (none) -> AC0805FR-7W100RL; Manufacturer (none) -> YAGEO; Package (none) -> 0805
- U1: MPN (none) -> MCP3208-CI/SL; Manufacturer (none) -> Microchip; Package (none) -> SOIC-16
- U10: MPN (none) -> ST485EBDR; Manufacturer (none) -> ST; Package (none) -> SOIC-8
Connections:
- net Sensor Module Prototype/ADC_TEMP_PT_1000: no longer U1.2 (CH1)
- net Sensor Module Prototype/INPUT_PT1000+: no longer J4.1 (Pin_1)
- net Sensor Module Prototype/INPUT_PT1000-: no longer J4.2 (Pin_2)
- new net ANALOG_GND: R4.2
- new net DIGITAL_GND: R4.1
- no-connect marks 1 -> 4
Other:
- added sheet Harness (Harness.kicad_sch)
- note added: "AGND and DGND are tied together internally to the MCP320X. This connection should be as close to thay chip as possible."
- note added: "ERC Overrides"
- note added: "RS-485 transceiver: Using Cat5 cable, the characteristic impedance is 100 Ohm. Adding a DC termination resistor of 100 Ohm to both ends of the cable should suffice for termination. This adds a DC load to the drivers though and you should consider designing an AC termination instead (Rt in series with a cap -- this messes up the rise and fall times though so you have to do it carefully)."
- note removed: "Using Cat5 cable, the characteristic impedance is 100 Ohm. Adding a DC termination resistor of 100 Ohm to both ends of the cable should suffice for termination. This adds a DC load to the drivers though and you should consider designing an AC termination instead (Rt in series with a cap -- this messes up the rise and fall times though so you have to do it carefully)."
