File: sensor_module_4.kicad_sch (KiCad schematic)
At the start: 42 parts, among them J18 EZO Carrier Board, J6 Cal_in, U15 TLV4387, U9 TLV2387DR

Commit message: feature/v3.1/setup - Inception - some general changes in support of v3.1 before I thought to branch.
Parts:
- C17, C2, C23, C24, C25, C5: MPN (none) -> CC0805KKX7R7BB824; Manufacturer (none) -> YAGEO; Package (none) -> 0805
- C3: MPN (none) -> CC0805KKX7R7BB824; Manufacturer (none) -> YAGEO; Package (none) -> 0805; now not fitted; now left out of the parts list
- C31, C48, C91: MPN (none) -> CL21B105KOFNNNG; Manufacturer (none) -> Samsung; Package (none) -> 0805
- C32, C4, C46, C58, C92: MPN (none) -> CC0805KRX7R7BB104; Manufacturer (none) -> YAGEO; Package (none) -> 0805
- D10: MPN (none) -> PTVS5V0Z1USK; Manufacturer (none) -> Nexperia; Package (none) -> DSN1608-2
- J18: now not fitted
- R1, R19, R20, R24, R36, R8: MPN (none) -> AC0805FR-7W1KL; Manufacturer (none) -> YAGEO; Package (none) -> 0805
- R10, R37, R7: MPN (none) -> AC0805FR-7W1KL; Manufacturer (none) -> YAGEO; Package (none) -> 0805; now not fitted; now left out of the parts list
- R11, R2, R3: MPN (none) -> AC0805FR-7W100KL; Manufacturer (none) -> YAGEO; Package (none) -> 0805
- R12: MPN (none) -> AC0805FR-7W10KL; Manufacturer (none) -> YAGEO; Package (none) -> 0805
- R17, R21: MPN (none) -> AC0805FR-7W10KL; Manufacturer (none) -> YAGEO; Package (none) -> 0805; now not fitted; now left out of the parts list
- R18: MPN (none) -> RCC0805470RFKEA; Manufacturer (none) -> Vishay-Dale; Package (none) -> 0805
- R22: MPN (none) -> AC0805FR-7W4K7L; Manufacturer (none) -> YAGEO; Package (none) -> 0805
- R23, R35: MPN (none) -> RC0805FR-7W27KL; Manufacturer (none) -> YAGEO; Package (none) -> 0805; now not fitted; now left out of the parts list
- R25: value 96k / 1% -> 91k / 1%; MPN (none) -> AC0805FR-7W91KL; Manufacturer (none) -> YAGEO; Package (none) -> 0805
- R26, R6: MPN (none) -> AC0805FR-7W100RL; Manufacturer (none) -> YAGEO; Package (none) -> 0805
- U15: MPN (none) -> TLV4387PWR; Manufacturer (none) -> TI; Package (none) -> TSSOP-14
- U9: MPN (none) -> TLV2387DR; Manufacturer (none) -> TI; Package (none) -> SOIC-8
Connections:
- net at R17.2: no longer U9.5 (+)
- net at R21.1, R35.1: no longer U9.6 (-)
- net at R23.2, R35.2, R37.1: no longer U9.7
Other:
- note added: "Note that the Atlas Scientific DO board is simply a 5-3.3V regulator coupled with a non-inverting amp with 10x gain on it. 100% saturation is 42mV out of the A.S. board so I'm assuming the probe outputs a max of 4.2mV. We will simply use a 910X gain stage here giving us very nearly full scale at 100% saturation. GAIN = 91k"
- note removed: "Note that the Atlas Scientific DO board is simply a 5-3.3V regulator coupled with a non-inverting amp with 10x gain on it. 100% saturation is 42mV out of the A.S. board so I'm assuming the probe outputs a max of 4.2mV. We will simply use a 960X gain stage here giving us very nearly full scale at 100% saturation. GAIN = 960x"
- moved on the sheet: U9B
